Commit message: diff_controller

File: robot_description/urdf/warehouse_r2d2.urdf.xacro (robot description, xacro)
@@ -2,4 +2,5 @@
 <robot name="r2d2"
        xmlns:xacro="http://www.ros.org/wiki/xacro">
+    <xacro:arg name="controllers_file" default=""/>
   <material name="blue">
     <color rgba="0 0 0.8 1"/>
@@ -290,3 +291,41 @@
         velocity="1.0"/>
 </joint>
+<ros2_control name="GazeboSystem" type="system">
+    <hardware>
+        <plugin>gazebo_ros2_control/GazeboSystem</plugin>
+    </hardware>
+    <joint name="left_front_wheel_joint">
+        <command_interface name="velocity"/>
+        <state_interface name="position"/>
+        <state_interface name="velocity"/>
+    </joint>
+    <joint name="left_back_wheel_joint">
+        <command_interface name="velocity"/>
+        <state_interface name="position"/>
+        <state_interface name="velocity"/>
+    </joint>
+    <joint name="right_front_wheel_joint">
+        <command_interface name="velocity"/>
+        <state_interface name="position"/>
+        <state_interface name="velocity"/>
+    </joint>
+    <joint name="right_back_wheel_joint">
+        <command_interface name="velocity"/>
+        <state_interface name="position"/>
+        <state_interface name="velocity"/>
+    </joint>
+    <joint name="head_swivel">
+        <command_interface name="position"/>
+        <state_interface name="position"/>
+        <state_interface name="velocity"/>
+    </joint>
+</ros2_control>
+<gazebo>
+    <plugin name="gazebo_ros2_control"
+            filename="libgazebo_ros2_control.so">
+        <robot_param>robot_description</robot_param>
+        <robot_param_node>robot_state_publisher</robot_param_node>
+        <parameters>$(arg controllers_file)</parameters>
+    </plugin>
+</gazebo>
 </robot>
